File: Hardware/TestRig.sch (EAGLE design)
At the start: 15 parts

Commit message: git ignore
Parts:
- added C1, C2, C4, C5: 1.0uF, SparkFun-Capacitors:1.0UF-25V-+80/-20(0805)
- added C3, C6: 0.1uF, SparkFun-Capacitors:0.1UF-25V(+80/-20%)(0603)
- added JP12: USBSMD, SparkFun-Connectors:USBSMD
- added U1: MIC5219 3.3V, SparkFun-PowerIC:V_REG_MIC52193.3V
Connections:
- new net VIN: C4.1, C5.1, C6.1, JP12.VBUS, U1.EN, U1.IN
- net GND: now also C1.2, C2.2, C3.2, C4.2, C5.2, C6.2, JP12.GND, U1.GND
- net VCC: now also C1.1, C2.1, C3.1, U1.OUT
Other:
- moved on the sheet: E_1_BASIC, E_1_GPIO, E_1_I2C_1, E_1_I2C_6, E_1_I2S, E_1_SD, E_1_SPI, E_1_UART_1, E_1_UART_2, E_1_USB, JP1, JP10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
