File: Hardware/TestRig.brd (EAGLE design)
At the start: 101.6 x 35.6 mm, 15 parts

Commit message: git ignore
Parts:
- added C1, C2, C4, C5: 1.0uF, SparkFun-Capacitors:0805
- added C3, C6: 0.1uF, SparkFun-Capacitors:0603-CAP
- added JP12: USBSMD, SparkFun-Connectors:USB-MINIB
- added U1: MIC5219 3.3V, SparkFun-PowerIC:SOT23-5
Connections:
- new net VIN: C4.1, C5.1, C6.1, JP12.VBUS, U1.1, U1.3
- net GND: now also C1.2, C2.2, C3.2, C4.2, C5.2, C6.2, JP12.GND, U1.2
- net VCC: now also C1.1, C2.1, C3.1, U1.5
Routing:
- added copper zone on layer 16, net VCC
- added copper zone on layer 16, net VIN
Other:
- board text added: "VCC 3.3v-4.5v"
Changed lines of the file:
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@@
 <setting verticaltext="up"/>
 </settings>
-<grid distance="0.025" unitdist="inch" unit="inch" style="lines" multiple="1" display="yes" altdistance="0.005" altunitdist="inch" altunit="inch"/>
+<grid distance="0.01" unitdist="inch" unit="inch" style="lines" multiple="1" display="yes" altdistance="0.005" altunitdist="inch" altunit="inch"/>
 <layers>
 <layer number="1" name="Top" color="4" fill="1" visible="yes" active="yes"/>
@@
 <rectangle x1="0" y1="21.59" x2="12.7" y2="35.56" layer="41"/>
 <text x="29.845" y="0.635" size="1.016" layer="21" font="vector" ratio="15" rot="R270" align="bottom-right">Edison BreadBoard Breakout</text>
+<text x="42.926" y="21.59" size="0.8128" layer="21" font="vector" ratio="15" rot="R180">VCC 3.3v-4.5v</text>
 </plain>
 <attributes>
@@
 <element name="LOGO1" library="SparkFun-Aesthetics" package="SFE_LOGO_NAME_FLAME_.1" value="SFE_LOGO_NAME_FLAME.1_INCH" x="5.715" y="22.86" rot="R90"/>
 <element name="LOGO2" library="SparkFun-Aesthetics" package="OSHW-LOGO-S" value="OSHW-LOGOS" x="3.175" y="3.175" rot="R90"/>
+<element name="U1" library="SparkFun-PowerIC" package="SOT23-5" value="MIC5219 3.3V" x="21.59" y="24.13" rot="MR90">
+<attribute name="PROD_ID" value="VREG-09872" x="21.59" y="24.13" size="1.778" layer="28" rot="MR90" display="off"/>
+</element>
+<element name="JP12" library="SparkFun-Connectors" package="USB-MINIB" value="USBSMD" x="19.05" y="30.48" rot="MR270">
+<attribute name="PROD_ID" value="CONN-08193" x="19.05" y="30.48" size="1.778" layer="28" rot="MR270" display="off"/>
+</element>
+<element name="C1" library="SparkFun-Capacitors" package="0805" value="1.0uF" x="24.765" y="24.13" rot="MR90">
+<attribute name="PROD_ID" value="CAP-11625" x="24.765" y="24.13" size="1.778" layer="28" rot="MR90" display="off"/>
+</element>
+<element name="C2" library="SparkFun-Capacitors" package="0805" value="1.0uF" x="26.67" y="24.13" rot="MR90">
+<attribute name="PROD_ID" value="CAP-11625" x="26.67" y="24.13" size="1.778" layer="28" rot="MR90" display="off"/>
+</element>
+<element name="C3" library="SparkFun-Capacitors" package="0603-CAP" value="0.1uF" x="28.575" y="24.13" rot="MR90">
+<attribute name="PROD_ID" value="CAP-00810" x="28.575" y="24.13" size="1.778" layer="28" rot="MR90" display="off"/>
+</element>
+<element name="C4" library="SparkFun-Capacitors" package="0805" value="1.0uF" x="18.415" y="24.765" rot="MR270">
+<attribute name="PROD_ID" value="CAP-11625" x="18.415" y="24.765" size="1.778" layer="28" rot="MR270" display="off"/>
+</element>
+<element name="C5" library="SparkFun-Capacitors" package="0805" value="1.0uF" x="16.51" y="24.765" rot="MR270">
+<attribute name="PROD_ID" value="CAP-11625" x="16.51" y="24.765" size="1.778" layer="28" rot="MR270" display="off"/>
+</element>
+<element name="C6" library="SparkFun-Capacitors" package="0603-CAP" value="0.1uF" x="14.605" y="24.765" rot="MR270">
+<attribute name="PROD_ID" value="CAP-00810" x="14.605" y="24.765" size="1.778" layer="28" rot="MR270" display="off"/>
+</element>
 </elements>
 <signals>
@@
 <via x="5.3848" y="19.1008" extent="1-16" drill="0.3302"/>
 <via x="7.1374" y="17.272" extent="1-16" drill="0.3302"/>
-<polygon width="0.1524" layer="16" spacing="0.254">
+<polygon width="0.1524" layer="16" spacing="0.254" rank="6">
 <vertex x="0" y="-0.05"/>
 <vertex x="31.75" y="-0.05"/>
@@
 <via x="4.699" y="17.3482" extent="1-16" drill="0.3302"/>
 <via x="4.0894" y="16.5862" extent="1-16" drill="0.3302"/>
+<contactref element="JP12" pad="GND"/>
+<contactref element="U1" pad="2"/>
+<contactref element="C1" pad="2"/>
+<contactref element="C2" pad="2"/>
+<contactref element="C3" pad="2"/>
+<contactref element="C4" pad="2"/>
+<contactref element="C6" pad="2"/>
+<contactref element="C5" pad="2"/>
 </signal>
 <signal name="3.3V">
@@
 <wire x1="10.922" y1="18.7452" x2="12.5984" y2="18.7452" width="0.8128" layer="1"/>
 <wire x1="12.5984" y1="18.7452" x2="16.9672" y2="23.114" width="0.8128" layer="1"/>
+<contactref element="U1" pad="5"/>
+<contactref element="C2" pad="1"/>
+<contactref element="C1" pad="1"/>
+<contactref element="C3" pad="1"/>
+<polygon width="0.254" layer="16">
+<vertex x="22.606" y="23.876"/>
+<vertex x="29.21" y="23.876"/>
+<vertex x="29.972" y="23.114"/>
+<vertex x="36.83" y="23.114"/>
+<vertex x="38.1" y="24.384"/>
+<vertex x="38.1" y="25.908"/>
+<vertex x="38.608" y="26.416"/>
+<vertex x="42.418" y="26.416"/>
+<vertex x="43.18" y="25.654"/>
+<vertex x="43.18" y="22.352"/>
+<vertex x="22.606" y="22.352"/>
+</polygon>
 </signal>
 <signal name="N$1">
@@
 <wire x1="52.07" y1="25.4508" x2="52.07" y2="25.4" width="0.1524" layer="1"/>
 </signal>
+<signal name="VIN">
+<contactref element="JP12" pad="VBUS"/>
+<contactref element="U1" pad="1"/>
+<contactref element="U1" pad="3"/>
+<contactref element="C4" pad="1"/>
+<contactref element="C6" pad="1"/>
+<contactref element="C5" pad="1"/>
+<polygon width="0.254" layer="16">
+<vertex x="19.812" y="23.368"/>
+<vertex x="19.812" y="23.114"/>
+<vertex x="21.336" y="23.114"/>
+<vertex x="21.336" y="26.416"/>
+<vertex x="18.034" y="26.416"/>
+<vertex x="18.034" y="29.464"/>
+<vertex x="15.748" y="29.464"/>
+<vertex x="15.748" y="26.416"/>
+<vertex x="14.224" y="26.416"/>
+<vertex x="14.224" y="25.146"/>
+<vertex x="21.082" y="25.146"/>
+<vertex x="21.082" y="23.368"/>
+</polygon>
+</signal>
 </signals>

Commit message: file cleanup
Routing:
- net N$19: track 67.9 -> 65.6 mm
