File: Hardware/Base_Block.sch (EAGLE design)
At the start: 46 parts, among them Q1 BSS138, U2 FTS31XS-U, U4 TPS62065

Commit message: added bottom side fids
Parts:
- added FID3, FID4: FIDUCIAL1X2, SparkFun-Aesthetics:FIDUCIAL1X2
Changed lines of the file:
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@@
 <part name="R15" library="SparkFun-Resistors" deviceset="1KOHM1/10W1%(0603)" device="" value="1K"/>
 <part name="SUPPLY7" library="SparkFun-Aesthetics" deviceset="5V" device=""/>
+<part name="FID3" library="SparkFun-Aesthetics" deviceset="FIDUCIAL" device="1X2"/>
+<part name="FID4" library="SparkFun-Aesthetics" deviceset="FIDUCIAL" device="1X2"/>
 </parts>
 <sheets>
@@
 <instance part="R15" gate="G$1" x="190.5" y="111.76" rot="R180"/>
 <instance part="SUPPLY7" gate="G$1" x="182.88" y="114.3"/>
+<instance part="FID3" gate="G$1" x="241.3" y="30.48"/>
+<instance part="FID4" gate="G$1" x="246.38" y="30.48"/>
 </instances>
 <busses>
